File: 单节锂电池板/Music_Player.kicad_pcb (KiCad board)
At the start: 4 copper layers, 28.3 x 23.8 mm, 40 parts, among them J1 Conn_01x02_PWR, J2 Conn_01x02_PWR, J3 Conn_01x02_PWR, J4 Conn_01x04_Female, J5 Conn_01x01_Female, J6 Conn_01x01_Female, J7 Conn_01x01_Female, Q1 Q_NMOS_DGS, Q2 Q_PMOS_DGS, U1 ME2807A35M3G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

Commit message: 第二次更新
美化了一点点，缩小了一些
Parts:
- added G***: LOGO, 项目3专用库:logo1-!smd, B.Cu at (17.2, 14.4)
- moved C11 1.98 mm to (11.2, 12.5), turned to 90 degrees
Routing:
- net GND: track 87.4 -> 91.2 mm
- net Net-(C3-Pad2): track 12.0 -> 14.8 mm
- net Net-(C5-Pad1): track 10.9 -> 8.21 mm
- net Net-(L1-Pad2): track 8.72 -> 9.40 mm
